File: madcatdb/madcatdb.kicad_pcb (KiCad board)
At the start: 2 copper layers, 1 part

Commit message: done (lol)
Parts:
- added C1: 100n, Capacitor_SMD:C_1206_3216Metric, F.Cu at (-8.30, 2.70)
- added F1: 500mA, Fuse:Fuse_1206_3216Metric, F.Cu at (-9.30, 9.70)
- added H1: M3, Crokto:M3_Via_Hole_NC, B.Cu at (-27.0, 3.50)
- added H2: M3_Pad, Crokto:M3_Via_Hole, F.Cu at (12.0, 3.50)
- added J1: USB_C_Receptacle_USB2.0, Crokto:USB_C_Receptacle_HRO_TYPE-C-31-M-12, F.Cu at (0.00, 0.00)
- added J2: Conn_01x04, Crokto:JST_SH_SM04B-SRSS-TB-Handsoldering, F.Cu at (-18.5, 3.92)
- added R1: 5.1k, Crokto:R_0603_1608Metric, F.Cu at (6.20, 5.60)
- added R2: 5.1k, Crokto:R_0603_1608Metric, F.Cu at (6.20, 9.07)
- added R3: 1M, Resistor_SMD:R_1206_3216Metric, F.Cu at (-10.7, 2.70)
- added U1: USBLC6-2SC6, Package_TO_SOT_SMD:SOT-23-6, F.Cu at (-10.7, 6.77)
- H3: renamed from H1; value JLCJLCJLCJLC -> jlc; moved to F.Cu
- moved H3 345.3 mm to (0.00, 4.60), turned to 180 degrees
Routing:
- net Earth: track 0.00 -> 41.9 mm
- net GND: track 0.00 -> 33.4 mm, vias 0 -> 5
- net DB+: track 0.00 -> 15.0 mm
- net DB-: track 0.00 -> 14.1 mm
- net VBUS: track 0.00 -> 13.8 mm, vias 0 -> 3
- net +5V: track 0.00 -> 13.2 mm, vias 0 -> 2
- net D-: track 0.00 -> 12.3 mm
- net D+: track 0.00 -> 12.3 mm
- net Net-(J1-PadB5): track 0.00 -> 9.51 mm, vias 0 -> 2
- net Net-(J1-PadA5): track 0.00 -> 9.11 mm
- added copper zone on B.Cu, net Earth
- added copper zone on F.Cu, net Earth
- added copper zone on B.Cu, net GND
Other:
- board outline added: 46 x 11 mm
