File: madcatdb/madcatdb.kicad_sch (KiCad schematic)
At the start: 11 parts, among them J1 USB_C_Receptacle_USB2.0, J2 Conn_01x04, U1 SRV05-4

Commit message: updated madcat to mid mount
Parts:
- J1: footprint Crokto:USB_C_Receptacle_HRO_TYPE-C-31-M-12 -> Crokto:HRO-TYPE-C-31-M-14
Changed lines of the file:
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@@
     (property "Reference" "J1" (id 0) (at 34.29 21.59 0))
     (property "Value" "USB_C_Receptacle_USB2.0" (id 1) (at 34.29 24.13 0))
-    (property "Footprint" "Crokto:USB_C_Receptacle_HRO_TYPE-C-31-M-12" (id 2) (at 38.1 44.45 0)
+    (property "Footprint" "Crokto:HRO-TYPE-C-31-M-14" (id 2) (at 38.1 44.45 0)
       (effects (font (size 1.27 1.27)) hide)
     )
@@
     )
     (path "/74f5ec08-7600-4a0b-a9e4-aae29f9ea08a"
-      (reference "J1") (unit 1) (value "USB_C_Receptacle_USB2.0") (footprint "Crokto:USB_C_Receptacle_HRO_TYPE-C-31-M-12")
+      (reference "J1") (unit 1) (value "USB_C_Receptacle_USB2.0") (footprint "Crokto:HRO-TYPE-C-31-M-14")
     )
     (path "/0471f253-a72b-4ea7-b6f0-5ec6d893951b"
