File: squatterboard2/squatterboard2.kicad_pcb (KiCad board)
At the start: 2 copper layers, 44 x 11 mm, 11 parts, among them J1 USB_C_Receptacle_USB2.0, J2 Conn_01x04, U1 SRV05-4

Commit message: added generic squatterboard2 version
Parts:
- H1: moved to F.Cu
- turned H1 to 0 degrees
Changed lines of the file:
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@@
     )
+  )
+  (footprint "Crokto:M3_Via_Hole_NC" (layer "F.Cu")
+    (at 3.5 3.5)
+    (descr "Mounting Hole 3.2mm, M3")
+    (tags "mounting hole 3.2mm m3")
+    (property "Sheetfile" "madcatdb.kicad_sch")
+    (property "Sheetname" "")
+    (attr exclude_from_pos_files)
+    (fp_text reference "H1" (at 0 -4.2) (layer "F.SilkS") hide
+      (effects (font (size 1 1) (thickness 0.15)))
+    )
+    (fp_text value "M3" (at 0 4.2) (layer "F.Fab")
+      (effects (font (size 1 1) (thickness 0.15)))
+    )
+    (fp_circle (center 0 0) (end 3.3 0) (layer "F.CrtYd") (width 0.1) (fill none))
+    (pad "" thru_hole circle (at -2.3 0) (size 0.8 0.8) (drill 0.5) (layers *.Cu "F.Mask"))
+    (pad "" thru_hole circle (at 1.626346 -1.626346) (size 0.8 0.8) (drill 0.5) (layers *.Cu "F.Mask"))
+    (pad "" thru_hole circle (at 1.626346 1.626346) (size 0.8 0.8) (drill 0.5) (layers *.Cu "F.Mask"))
+    (pad "" thru_hole circle (at 0 0) (size 6 6) (drill 3.2) (layers *.Cu "F.Mask"))
+    (pad "" thru_hole circle (at 0 2.3) (size 0.8 0.8) (drill 0.5) (layers *.Cu "F.Mask"))
+    (pad "" thru_hole circle (at 0 -2.3) (size 0.8 0.8) (drill 0.5) (layers *.Cu "F.Mask"))
+    (pad "" thru_hole circle (at -1.626346 1.626346) (size 0.8 0.8) (drill 0.5) (layers *.Cu "F.Mask"))
+    (pad "" thru_hole circle (at -1.626346 -1.626346) (size 0.8 0.8) (drill 0.5) (layers *.Cu "F.Mask"))
+    (pad "" thru_hole circle (at 2.3 0) (size 0.8 0.8) (drill 0.5) (layers *.Cu "F.Mask"))
   )
   (footprint "Capacitor_SMD:C_1206_3216Metric" (layer "F.Cu")
@@
     )
   )
-  (footprint "Crokto:M3_Via_Hole_NC" (layer "B.Cu")
-    (at 3.5 3.5 180)
-    (descr "Mounting Hole 3.2mm, M3")
-    (tags "mounting hole 3.2mm m3")
-    (property "Sheetfile" "madcatdb.kicad_sch")
-    (property "Sheetname" "")
-    (attr exclude_from_pos_files)
-    (fp_text reference "H1" (at 0 4.2) (layer "B.SilkS") hide
-      (effects (font (size 1 1) (thickness 0.15)) (justify mirror))
-    )
-    (fp_text value "M3" (at 0 -4.2) (layer "B.Fab")
-      (effects (font (size 1 1) (thickness 0.15)) (justify mirror))
-    )
-    (fp_circle (center 0 0) (end 3.3 0) (layer "B.CrtYd") (width 0.1) (fill none))
-    (pad "" thru_hole circle (at -2.3 0 180) (size 0.8 0.8) (drill 0.5) (layers *.Cu "B.Mask"))
-    (pad "" thru_hole circle (at 1.626346 1.626346 180) (size 0.8 0.8) (drill 0.5) (layers *.Cu "B.Mask"))
-    (pad "" thru_hole circle (at 1.626346 -1.626346 180) (size 0.8 0.8) (drill 0.5) (layers *.Cu "B.Mask"))
-    (pad "" thru_hole circle (at 0 0 180) (size 6 6) (drill 3.2) (layers *.Cu "B.Mask"))
-    (pad "" thru_hole circle (at 0 -2.3 180) (size 0.8 0.8) (drill 0.5) (layers *.Cu "B.Mask"))
-    (pad "" thru_hole circle (at 0 2.3 180) (size 0.8 0.8) (drill 0.5) (layers *.Cu "B.Mask"))
-    (pad "" thru_hole circle (at -1.626346 -1.626346 180) (size 0.8 0.8) (drill 0.5) (layers *.Cu "B.Mask"))
-    (pad "" thru_hole circle (at -1.626346 1.626346 180) (size 0.8 0.8) (drill 0.5) (layers *.Cu "B.Mask"))
-    (pad "" thru_hole circle (at 2.3 0 180) (size 0.8 0.8) (drill 0.5) (layers *.Cu "B.Mask"))
-  )
   (gr_arc (start 2 11) (mid 0.585786 10.414214) (end 0 9) (layer "Edge.Cuts") (width 0.1))
